Commit message: ฅ^•ﻌ•^ฅ

File: Module6/ex03/src/robot_description/urdf/gazebo.urdf.xacro (robot description, xacro)
@@ -50,5 +50,5 @@
         </plugin>
         <plugin filename="gz-sim-imu-system"
-        	name="gz::sim::systems::Imu">
+        name="gz::sim::systems::Imu">
         </plugin>
     </gazebo>

File: Module6/ex03/src/robot_description/urdf/imu.urdf.xacro (robot description, xacro)
@@ -1,8 +1,6 @@
 <?xml version="1.0"?>
 <robot xmlns:xacro="http://www.ros.org/wiki/xacro" name="imu">
-    <xacro:property name="height" value="0.65"/>
-    <xacro:property name="block_thickness" value="0.05"/>
     <joint name="imu_sensor_joint" type="fixed">
-        <origin xyz="0 0 ${8 * height / 12 + 0.05}"/>
+        <origin xyz="0.11 0.05 0.05" rpy="0 0 0"/>
         <parent link="base_link"/>
         <child link="imu_sensor_link"/>
@@ -10,15 +8,21 @@
     <link name="imu_sensor_link">
         <inertial>
+        <origin xyz="0 0 0" rpy="0 0 0"/>
         <mass value="0.02" />
-        <inertia ixx="${(1/12) * 0.02 * 2 * (0.05*0.05)}" ixy="0.0" ixz="0.0"
-                 iyy="${(1/12) * 0.02 * (0.02*0.02+0.05*0.05)}" iyz="0.0"
-                 izz="${(1/12) * 0.02 * (0.02*0.02+0.05*0.05)}" />
+        <inertia ixx="${(1/12) * 0.01 * (0.2*0.2+0.5*0.5)}" ixy="0.0" ixz="0.0"
+                 iyy="${(1/12) * 0.01 * (0.2*0.2+0.5*0.5)}" iyz="0.0"
+                 izz="${(1/12) * 0.01 * (0.2*0.2+0.5*0.5)}" />
     </inertial>
     <visual>
+        <origin xyz="0 0 0"/>
         <geometry>
             <box size="0.02 0.05 0.05"/>
         </geometry>
+        <material name="Grey1">
+			<color rgba="0.2 0.1 0.0 1.0"/>
+		</material>
     </visual>
     <collision>
+        <origin xyz="0 0 0"/>
         <geometry>
             <box size="0.02 0.05 0.05"/>
@@ -29,9 +33,8 @@
         <gravity>true</gravity>
         <sensor name='imu_sensor' type='imu'>
-            <!-- важно! -->
-            <gz_frame_id>robot/imu_sensor_link</gz_frame_id>
             <always_on>true</always_on>
-            <update_rate>0,5</update_rate>
+            <update_rate>1</update_rate>
             <visualize>true</visualize>
+            <topic>imu</topic>
             <pose>0 0 0 0 0 0</pose>
         </sensor>

File: Module6/ex03/src/robot_description/urdf/robot_lab6.urdf.xacro (robot description, xacro)
@@ -4,5 +4,5 @@
     <xacro:include filename="$(find robot_description)/urdf/robot_lidar.urdf.xacro" />
     <xacro:include filename="$(find robot_description)/urdf/depth.urdf.xacro" />
-    <xacro:include filename="$(find robot_description)/urdf/imu.urdf.xacro" />
+    <xacro:include filename="imu.urdf.xacro" />
     <!-- Robot properites -->
     <xacro:property name="base_width" value="0.31"/>
@@ -189,11 +189,3 @@
         <mu2 value="0.001"/>
     </gazebo>
-    <gazebo reference="link_chassis">
-    	<sensor name="imu_sensor" type="imu">
-    		<always_on>1</always_on>
-    		<update_rate>20</update_rate>
-    		<visualize>true</visualize>
-    		<topic>imu</topic>
-    	</sensor>
-    </gazebo>
 </robot>
